File: Watchy.sch (KiCad schematic (older format))
At the start: 55 parts, among them J1 FPC24(0.5MM), J2 Micro USB, J3 Battery, M1 Vibration_Motor, Q1 AO3400A, Q2 UMH3N, Q4 CJ2301, Q5 S8050, SW1 BTN, SW2 BTN, SW3 BTN, SW4 BTN, U1 ESP32-PICO-D4, U2 ME6211C33M5G-N, U3 CP2104, U4 BMA423, U5 TP4054, U6 DS3231MZ

Commit message: Modifications done during livestream 18th January 2021 for a schmartwatch 2.0 based on the Watchy
- Use DCDC switch mode power supply
- Change RTC to RV-3028
- Use a chip antenna for BLE/WiFi connection
- Review of e-Paper connector for 3 color e-ink
- Forward annotation and initial placing done for PCB
Parts:
- removed AE1: SWRA117D, Watchy:SWRA117D, symbol Device:Antenna_Chip
- removed J2: Micro USB, Watchy:USB_Micro-B, symbol Connector:USB_OTG
- removed L1: 10uH 1A, Inductors:Inductor_Taiyo-Yuden_NR-40xx, symbol Device:L
- removed Q4: CJ2301, TO_SOT_Packages_SMD:SOT-23, symbol Transistor_FET:BSS83P
- removed U2: ME6211C33M5G-N, TO_SOT_Packages_SMD:SOT-23-5, symbol Regulator_Linear:TLV70033_SOT23-5
- removed U4: BMA423, Housings_LGA:LGA-12_2x2mm_Pitch0.5mm, symbol Watchy:BMA423
- removed U6: DS3231MZ, Housings_SOIC:SOIC-8_3.9x4.9mm_Pitch1.27mm, symbol Timer_RTC:DS3231MZ
- added AE1: Antenna_Chip, Watchy:ANT_ANT016008LCS2442MA2, symbol Watchy:Antenna_Chip
- added C13, C16: 100nF, Capacitor_SMD:C_0603_1608Metric, symbol Device:C
- added C15: 4.7uF/50V, Capacitor_SMD:C_0805_2012Metric, symbol Device:C
- added L1, L2: 2u2H, Inductor_SMD:L_0603_1608Metric, symbol Device:L_Small
- added L3: 2nH, Inductor_SMD:L_0402_1005Metric, symbol Device:L_Small
- added L4: 3nH, Inductor_SMD:L_0402_1005Metric, symbol Device:L_Small
- added P?: USB_C_Plug_USB2.0, Connector_USB:USB_C_Receptacle_Palconn_UTC16-G, symbol Connector:USB_C_Plug_USB2.0
- added Q3: CJ2301, Package_TO_SOT_SMD:SOT-23, symbol Transistor_FET:BSS83P
- added R11: 430k, Resistor_SMD:R_0402_1005Metric, symbol Device:R
- added R18, R19: 10K, Resistor_SMD:R_0402_1005Metric, symbol Device:R
- added U2: MT3420C, Package_TO_SOT_SMD:SOT-23-6, symbol Watchy:MT3420C
- added U4: LSM6DSOXTR, Watchy:PQFN50P250X300X86-14N, symbol Watchy:LSM6DSOXTR
- added U6: RV-3028-C7, Watchy:IC_RV-3028-C7, symbol Watchy:RV-3028-C7
- C12: value 4.7uF/50V -> 1uF/50V; footprint Capacitors_SMD:C_0805 -> Capacitor_SMD:C_0603_1608Metric
- C3, C4: footprint Capacitors_SMD:C_0805 -> Capacitor_SMD:C_0805_2012Metric
- D1, D2, D3, D4: footprint Diodes_SMD:D_SOD-123 -> Diode_SMD:D_SOD-123
- D5: footprint LEDs:LED_0603 -> LED_SMD:LED_0603_1608Metric
- M1: MPN (none) -> C1026B002F
- Q1, Q5: footprint TO_SOT_Packages_SMD:SOT-23 -> Package_TO_SOT_SMD:SOT-23
- Q2: footprint TO_SOT_Packages_SMD:SOT-363_SC-70-6 -> Package_TO_SOT_SMD:SOT-363_SC-70-6
- R1, R10, R12, R13, R14, R16, R17, R2, R3, R4, R5, R6, R7, R8, R9: footprint Resistors_SMD:R_0402 -> Resistor_SMD:R_0402_1005Metric
- R15: value 10K -> 100K; footprint Resistors_SMD:R_0402 -> Resistor_SMD:R_0402_1005Metric
- U1: footprint Housings_DFN_QFN:QFN-48-1EP_7x7mm_Pitch0.5mm -> Package_DFN_QFN:QFN-48-1EP_7x7mm_P0.5mm_EP5.45x5.45mm
- U5: footprint TO_SOT_Packages_SMD:SOT-23-5 -> Package_TO_SOT_SMD:SOT-23-5
Connections:
- wire segments 39 -> 70
- no-connect marks 40 -> 21
Other:
- note added: "Battery Charger"
- note added: "Display Power Supply"
- note added: "E-Paper Connector"
- note removed: "E-Paper Driver"
- moved on the sheet: C1, C10, C11, C14, C2, C3, C4, C5, C6, C7, C8, C9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
